Commit message: Uses hard-coded PLA density

File: robot.urdf (robot description, URDF)
Before this commit: robot my_robot, 0 links, 3 joints
Links:
- added link Foot_V2, mass 0.074616; collision mesh filename=package://my_robot/meshes/Foot_V2.stl; visual mesh filename=package://my_robot/meshes/Foot_V2.stl
- added link STS3125, mass 0.044802; collision mesh filename=package://my_robot/meshes/STS3125.stl; visual mesh filename=package://my_robot/meshes/STS3125.stl
- added link Servo_Case_to_Grid, mass 0.022553; collision mesh filename=package://my_robot/meshes/Servo_Case_to_Grid.stl; visual mesh filename=package://my_robot/meshes/Servo_Case_to_Grid.stl
Joints:
- joint STS3125_to_Foot_V2: origin xyz=0.000000 0.018000 -0.000000 rpy=0.000000 -0.000000 -1.570796 -> xyz=-0.000000 0.018000 -0.000000 rpy=0.000000 -0.000000 -1.570796
